File: KiCAD/RVController/RVController.kicad_sch (KiCad schematic)
At the start: 1 part, among them U1 FREESOC_MINI

Commit message: Getting started
Added GaN NFET output channels, started work on input channels
Parts:
- added C1: 10UF, Capacitor_SMD:C_1206_3216Metric, symbol Device:C
- added C2: 100u, Capacitor_THT:CP_Radial_D8.0mm_P3.50mm, symbol Device:C
- added C3, C? (x2): 100u, Capacitor_THT:CP_Radial_D6.3mm_P2.50mm, symbol Device:C
- added D? (x8): D_Schottky, symbol Device:D_Schottky
- added J1, J2, J3, J4: 1727078, PHOENIX_1727078, symbol Schematic:1727078
- added J? (x2): Conn_01x02_Male, symbol Connector:Conn_01x02_Male
- added Q1, Q2, Q3, Q4, Q5, Q6, Q7, Q8: EPC2014C, TRANS_EPC2014C, symbol Schematic:EPC2014C
- added R? (x3): 1k, symbol Device:R
- added R?: 22k, symbol Device:R
- added R? (x2): 4.7k, symbol Device:R
- added U2: 74HCT541, Package_DIP:DIP-20_W7.62mm_LongPads, symbol 74xx:74HCT541
- added U3: VX7805-500, Footprints:VX78012-500_VX7805-500, symbol Schematic:VX7805-500
Connections:
- net GND: now reaches U1.20 (GND)
- net GND: now also C1.2, C2.2, C3.2, C?.2, C?.2, D?.2 (A), D?.2 (A), D?.2 (A), J2.2, J2.4, J2.6, J2.8, J4.2, J4.4, J4.6, J4.8, Q1.2, Q1.4, Q2.2, Q2.4, Q3.2, Q3.4, Q4.2, Q4.4, Q5.2, Q5.4, Q6.2, Q6.4, Q7.2, Q7.4, Q8.2, Q8.4, R?.2, R?.2, U2.1 (G1), U2.10 (GND), U2.19 (G2), U3.2 (GND/-VOUT)
- net XPWM1: now reaches U1.21 (2.0)
- net XPWM1: now also U2.2 (A0)
- net XPWM2: now reaches U1.22 (2.1)
- net XPWM2: now also U2.3 (A1)
- net XPWM3: now reaches U1.23 (2.2)
- net XPWM3: now also U2.4 (A2)
- net XPWM4: now reaches U1.24 (2.3)
- net XPWM4: now also U2.5 (A3)
- net XPWM5: now reaches U1.25 (2.4)
- net XPWM5: now also U2.6 (A4)
- net XPWM6: now reaches U1.26 (2.5)
- net XPWM6: now also U2.7 (A5)
- net XPWM7: now reaches U1.27 (2.6)
- net XPWM7: now also U2.8 (A6)
- net XPWM8: now reaches U1.28 (2.7)
- net XPWM8: now also U2.9 (A7)
- net ADC1: now reaches U1.39 (0.0)
- net ADC1: now also D?.1 (K), D?.2 (A), J?.1 (Pin_1), R?.1, R?.2
- net +5V: now reaches U1.40 (VDD)
- net +5V: now also C1.1, C3.1, D?.1 (K), D?.1 (K), D?.1 (K), R?.1, U2.20 (VCC), U3.3 (+VOUT/GND)
- new net: C?.1, J?.2 (Pin_2) (x2)
- new net: D?.1 (K), D?.2 (A), R?.2, R?.2
- new net ADC2: D?.1 (K), D?.2 (A), J?.1 (Pin_1), R?.1, R?.2
- new net INPUT1: D?.2 (A), J2.1, R?.1
- new net INPUT2: D?.2 (A), J2.3, R?.1, R?.1
- new net INPUT3: J2.5
- new net INPUT4: J2.7
- new net INPUT5: J4.1
- new net INPUT6: J4.3
- new net INPUT7: J4.5
- new net INPUT8: J4.7
- new net LED1: J1.2, Q1.3, Q1.5
- new net LED2: J1.4, Q2.3, Q2.5
- new net LED3: J1.6, Q3.3, Q3.5
- new net LED4: J1.8, Q4.3, Q4.5
- new net LED5: J3.2, Q5.3, Q5.5
- new net LED6: J3.4, Q6.3, Q6.5
- new net LED7: J3.6, Q7.3, Q7.5
- new net LED8: J3.8, Q8.3, Q8.5
- new net PWM1: Q1.1, U2.18 (Y0)
- new net PWM2: Q2.1, U2.17 (Y1)
- new net PWM3: Q3.1, U2.16 (Y2)
- new net PWM4: Q4.1, U2.15 (Y3)
- new net PWM5: Q5.1, U2.14 (Y4)
- new net PWM6: Q6.1, U2.13 (Y5)
- new net PWM7: Q7.1, U2.12 (Y6)
- new net PWM8: Q8.1, U2.11 (Y7)
- new net VBUS: C2.1, D?.1 (K), D?.1 (K), J1.1, J1.3, J1.5, J1.7, J3.1, J3.3, J3.5, J3.7, U3.1 (+VIN)
Other:
- note added: "Vout = 1/5.7 Vin 12Vin = 2.1Vout @ 2mA 24Vin = 4.2Vout @ 4mA"
- moved on the sheet: U1
