File: KiCAD/RVController/RVController.kicad_sch (KiCad schematic)
At the start: 81 parts, among them IC1 MCP2561FD-E/P, J1 1727078, J10 Conn_01x02_Male, J11 Conn_01x02_Male, J12 284392-2, J2 1727078, J3 1727078, J4 1727078, J5 4-1437652-0, J6 Conn_01x02_Male, J7 Conn_01x02_Male, J8 54602-908LF, J9 54602-908LF, U1 114-83-640-41-134161, U2 74HCT541, U3 VX7805-500, U4 H11L1SR2M, U5 H11L1SR2M, Y1 ECS-3961-240-AU-TR

Commit message: Updates to new parts, routed
Changed to alternative FETs, Schottky diodes, TVS, etc. Ready for production
Parts:
- removed C3: C, Capacitor_THT:CP_Radial_D6.3mm_P2.50mm, symbol Device:C
- removed C4, C5: 100u, Capacitor_THT:CP_Radial_D6.3mm_P2.50mm, symbol Device:C
- removed C7: 10UF, Capacitor_SMD:C_1206_3216Metric, symbol Device:C
- removed C8: 4700pF, Capacitor_SMD:C_0603_1608Metric, symbol Device:C
- removed D1, D10, D11, D12, D17, D18, D19, D2, D20, D3, D4, D5, D6, D7, D8, D9: SS16MH, Footprints:SODFL2512X73N, symbol Schematic:SS16MH
- removed D13, D15: ATV02W240B, Diode_SMD:D_SOD-123FAC, symbol Schematic:SS16MH
- removed IC1: MCP2561FD-E/P, Package_DIP:DIP-8_W7.62mm_LongPads, symbol Schematic:MCP2561FD-E/P
- removed J1, J2, J3, J4: 1727078, PHOENIX_1727078, symbol Schematic:1727078
- removed J10, J11, J6, J7: Conn_01x02_Male, Connector_PinHeader_2.54mm:PinHeader_1x02_P2.54mm_Vertical, symbol Connector:Conn_01x02_Male
- removed J12: 284392-2, Footprints:TE_284392-2, symbol Schematic:284392-2
- removed J8, J9: 54602-908LF, Footprints:AMPHENOL_54602-908LF, symbol Schematic:54602-908LF
- removed R1, R11, R12, R13, R2, R26, R28, R3: 1K, Resistor_SMD:R_0805_2012Metric, symbol Device:R
- removed R14, R15, R16, R4, R5, R6: 22K, Resistor_SMD:R_0805_2012Metric, symbol Device:R
- removed R17, R22, R23: 300R, Resistor_SMD:R_0805_2012Metric, symbol Device:R
- removed R24, R29: 60R, Resistor_SMD:R_0805_2012Metric, symbol Device:R
- removed R25, R27: 4.7K, Resistor_SMD:R_0805_2012Metric, symbol Device:R
- removed U3: VX7805-500, Footprints:VX78012-500_VX7805-500, symbol Schematic:VX7805-500
- removed U4, U5: H11L1SR2M, Footprints:IC_H11L1SR2M, symbol Schematic:H11L1SR2M
- added C2, C3, C4, C8: 1206,100nF,50V,X7R, Capacitor_SMD:C_1206_3216Metric, symbol jlcpcb-basic-capacitor:1206,100nF,50V,X7R
- added C7, C9: 1206,1uF,50V,X7R, Capacitor_SMD:C_1206_3216Metric, symbol jlcpcb-basic-capacitor:1206,1uF,50V,X7R
- added P1, P2, P3, P4, P5, P6, P7, P8: WJ124-3_81-4P, Footprints:CONN-TH_4P-P3.81_KF124-3.81-4P, symbol Schematic:WJ124-3_81-4P
- added S1: MSDR-16S, Footprints:SW-SMD_6P-L7.4-W7.4-P2.54-LS9.5-TL, symbol Schematic:MSDR-16S
- added U2: CJ7805_3%, Package_TO_SOT_SMD:TO-252-2, symbol Schematic:CJ7805_3%
- C1: renamed from C2; value 100u -> HZA107M050G24T-F; footprint Capacitor_THT:CP_Radial_D8.0mm_P3.50mm -> Capacitor_SMD:CP_Elec_10x10; symbol Device:C -> Device:C_Polarized; PN EEH-AZF1V101B -> HZA107M050G24T-F; Voltage 35V -> 50V
- J1: renamed from J5; footprint TE_4-1437652-0 -> Footprints:TE_4-1437652-0; PN HB9500-9.5-2P -> C60785
- U3: renamed from U2; value 74HCT541 -> C554416; footprint Package_DIP:DIP-20_W7.62mm_LongPads -> Package_SO:SOIC-20W_7.5x12.8mm_P1.27mm; PN CD74ACT541EE4 -> C554416
- renumbered C1 to C5, R7 to R1, R8 to R2, R9 to R3, R10 to R4, R18 to R5, R19 to R6, R20 to R7, R21 to R8
Connections:
- net +5V_CAN is gone; now on net +5V: C6.1
- net GND_CAN is gone; now on net GND: C6.2
- net +5V: now also C2.1, C3.1, C8.1, U2.3 (Out)
- net GND: now also C2.2, C3.2, C4.2, C7.1, C8.2, C9.1, S1.C, U2.2 (GND)
- net INPUT1: now also P3.1
- net INPUT2: now also P3.3
- net INPUT3: now also P4.1
- net INPUT4: now also P4.3
- net INPUT5: now also P7.1
- net INPUT6: now also P7.3
- net INPUT7: now also P8.1
- net INPUT8: now also P8.3
- net LED1: now also P1.2
- net LED2: now also P1.4
- net LED3: now also P2.2
- net LED4: now also P2.4
- net LED5: now also P5.2
- net LED6: now also P5.4
- net LED7: now also P6.2
- net LED8: now also P6.4
- net VBUS: now also C4.1, P1.1, P1.3, P2.1, P2.3, P5.1, P5.3, P6.1, P6.3, U2.1 (IN)
- net at R5.2: now also P7.2
- net at R6.2: now also P7.4
- net at R7.2: now also P8.2
- net at R8.2: now also P8.4
- net at R3.2: now also P4.2
- net at R4.2: now also P4.4
- net at R1.2: now also P3.2
- net ADDR_4: now reaches U1.31 (1.6)
- net ADDR_4: now also S1.4
- net ADDR_1: now reaches U1.32 (0.7)
- net ADDR_1: now also S1.1
- net ADDR_2: now reaches U1.33 (0.6)
- net ADDR_2: now also S1.2
- net ADDR_8: now reaches U1.34 (0.5)
- net ADDR_8: now also S1.8
- net at U1.35 (0.4): now also C7.2
- net at U1.37 (0.2): now also C9.2
- net at R2.2: now also P3.4
- no-connect marks 25 -> 10
Other:
- added sheet CAN (can_interface.kicad_sch)
- added sheet Inputs (inputs.kicad_sch)
- note removed: "Vout = 1/5.7 Vin 12Vin = 2.1Vout @ 2mA 24Vin = 4.2Vout @ 4mA"
- moved on the sheet: C5, J1, R1, R2, R3, R4, R5, R6, R7, R8, U1, U3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

Commit message: Production version
Connections:
- net GND: no longer Y1.1 (TRI-STATE)
Changed lines of the file:
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@@
     (pin "4")
-  )
-  (symbol (lib_id "power:GND") (at 35.56 76.2 0) (unit 1)
-    (in_bom yes) (on_board yes) (fields_autoplaced)
-    (property "Reference" "#PWR04" (id 0) (at 35.56 82.55 0)
-      (effects (font (size 1.27 1.27)) hide)
-    )
-    (property "Value" "GND" (id 1) (at 35.56 81.28 0))
-    (property "Footprint" "" (id 2) (at 35.56 76.2 0)
-      (effects (font (size 1.27 1.27)) hide)
-    )
-    (property "Datasheet" "" (id 3) (at 35.56 76.2 0)
-      (effects (font (size 1.27 1.27)) hide)
-    )
-    (pin "1")
   )
   (symbol (lib_id "Mechanical:MountingHole") (at 335.28 229.87 0) (unit 1)
@@
       (reference "#PWR03") (unit 1) (value "+5V") (footprint "")
     )
-    (path "/bbe4ce6b-0abf-4fdf-94bb-f50249d7d217"
-      (reference "#PWR04") (unit 1) (value "GND") (footprint "")
-    )
     (path "/6b269d09-32a8-4c94-9eeb-9c234b90b040"
