File: KiCAD/RVController/RVController.kicad_pcb (KiCad board)
At the start: 2 copper layers, 227.2 x 53 mm, 119 parts, among them IC1 TJA1042T/1J, J1 4-1437652-0, J2 284392-2, J3 54602-908LF, J4 54602-908LF, P1 WJ124-3_81-4P, P2 WJ124-3_81-4P, P3 WJ124-3_81-4P, P4 WJ124-3_81-4P, P5 WJ124-3_81-4P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

Commit message: Production version
Connections:
- Y1 pad 1: GND -> unconnected-(Y1-Pad1)
Routing:
- net GND: track 126.2 -> 119.5 mm
Changed lines of the file:
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@@
   (net 98 "/ADDR_4")
   (net 99 "/ADDR_8")
+  (net 100 "unconnected-(Y1-Pad1)")
   (footprint "Footprints:114-83-640-41-134161" (layer "F.Cu")
     (at 57.785 86.36 90)
@@
     (fp_circle (center -3 1.2) (end -2.9 1.2) (layer "F.Fab") (width 0.2) (fill none))
     (pad "1" smd rect (at -1.27 1.1 180) (size 1.4 1.2) (layers "F.Cu" "F.Paste" "F.Mask")
-      (net 20 "GND") (pinfunction "TRI-STATE") (pintype "input"))
+      (net 100 "unconnected-(Y1-Pad1)") (pinfunction "TRI-STATE") (pintype "input"))
     (pad "2" smd rect (at 1.27 1.1 180) (size 1.4 1.2) (layers "F.Cu" "F.Paste" "F.Mask")
       (net 20 "GND") (pinfunction "GND") (pintype "power_in"))
@@
   (segment (start 82.55 93.345) (end 81.915 93.98) (width 0.5) (layer "F.Cu") (net 20))
   (segment (start 105.361 80.01) (end 104.14 80.01) (width 0.5) (layer "F.Cu") (net 20))
-  (segment (start 33.147 100.541) (end 31.92 100.541) (width 0.5) (layer "F.Cu") (net 20))
   (segment (start 77.47 105.41) (end 77.47 107.0375) (width 0.5) (layer "F.Cu") (net 20))
   (segment (start 98.835 104.775) (end 99.695 104.775) (width 0.5) (layer "F.Cu") (net 20))
@@
   (segment (start 99.646 83.439) (end 97.663 83.439) (width 0.5) (layer "F.Cu") (net 20))
   (segment (start 136.1675 101.6) (end 138.43 101.6) (width 0.5) (layer "F.Cu") (net 20))
-  (segment (start 31.92 100.541) (end 31.291 101.17) (width 0.5) (layer "F.Cu") (net 20))
   (segment (start 139.065 102.235) (end 139.065 104.054854) (width 0.5) (layer "F.Cu") (net 20))
   (segment (start 84.455 104.775) (end 85.09 105.41) (width 0.5) (layer "F.Cu") (net 20))
@@
   (segment (start 153.3125 101.6) (end 155.575 101.6) (width 0.5) (layer "F.Cu") (net 20))
   (segment (start 66.42 104.775) (end 67.31 104.775) (width 0.5) (layer "F.Cu") (net 20))
-  (segment (start 33.147 100.541) (end 33.147 103.038854) (width 0.5) (layer "F.Cu") (net 20))
   (segment (start 145.6925 101.6) (end 147.955 101.6) (width 0.5) (layer "F.Cu") (net 20))
   (segment (start 67.945 105.41) (end 67.945 107.0375) (width 0.5) (layer "F.Cu") (net 20))
@@
   (segment (start 199.1525 93.013) (end 199.4845 93.345) (width 0.5) (layer "F.Cu") (net 20))
   (segment (start 156.21 102.235) (end 156.21 104.054854) (width 0.5) (layer "F.Cu") (net 20))
-  (segment (start 33.147 103.038854) (end 33.528 103.419854) (width 0.5) (layer "F.Cu") (net 20))
   (segment (start 90.346 82.169) (end 92.456 82.169) (width 0.5) (layer "F.Cu") (net 20))
   (segment (start 51.21 104.6425) (end 51.0775 104.775) (width 0.5) (layer "F.Cu") (net 20))
-  (segment (start 31.291 101.17) (end 29.718 101.17) (width 0.5) (layer "F.Cu") (net 20))
   (segment (start 76.835 104.775) (end 77.47 105.41) (width 0.5) (layer "F.Cu") (net 20))
   (segment (start 29.718 101.17) (end 29.718 102.997) (width 0.5) (layer "F.Cu") (net 20))
